File: speedctrl.sch (KiCad schematic (older format))
At the start: 18 parts, among them J1 Conn_02x04_Top_Bottom_Shielded, Q1 Q_NMOS_GSD, U2 BD6231, U3 LM317_3PinPackage

Commit message: Fix missing references
Parts:
- TR1: symbol speectrl_parts:ATB3225 -> speedctrl_parts:ATB3225
- U2: symbol speectrl_parts:BD6231 -> speedctrl_parts:BD6231
Connections:
- net labels removed: +16V
Changed lines of the file:
@@
 $EndDescr
 $Comp
-L speectrl_parts:BD6231 U2
+L speedctrl_parts:BD6231 U2
 U 1 1 5BA9883A
 P 8950 4150
@@
 F 3 "" H 8700 4500 50  0001 C CNN
 	1    8950 4150
-	1    0    0    -1
-$EndComp
-$Comp
-L speectrl_parts:+16V #PWR0101
-U 1 1 5BA98EB0
-P 8950 3650
-F 0 "#PWR0101" H 8950 3500 50  0001 C CNN
-F 1 "+16V" H 8965 3823 50  0000 C CNN
-F 2 "" H 8950 3650 50  0001 C CNN
-F 3 "" H 8950 3650 50  0001 C CNN
-	1    8950 3650
 	1    0    0    -1
 $EndComp
@@
 	9000 5950 9000 5900
 $Comp
-L speectrl_parts:ATB3225 TR1
+L speedctrl_parts:ATB3225 TR1
 U 1 1 5BB580A9
 P 9350 2000
@@
 Wire Wire Line
 	8950 1800 8950 1600
-$Comp
-L speectrl_parts:+16V #PWR0104
-U 1 1 5BB58AF7
-P 8950 1150
-F 0 "#PWR0104" H 8950 1000 50  0001 C CNN
-F 1 "+16V" H 8965 1323 50  0000 C CNN
-F 2 "" H 8950 1150 50  0001 C CNN
-F 3 "" H 8950 1150 50  0001 C CNN
-	1    8950 1150
-	1    0    0    -1
-$EndComp
 Wire Wire Line
 	8950 1300 8950 1150
@@
 Wire Wire Line
 	3600 4600 3800 4600
-$Comp
-L speectrl_parts:+16V #PWR?
-U 1 1 5BC2CCD6
-P 4800 4600
-F 0 "#PWR?" H 4800 4450 50  0001 C CNN
-F 1 "+16V" H 4815 4773 50  0000 C CNN
-F 2 "" H 4800 4600 50  0001 C CNN
-F 3 "" H 4800 4600 50  0001 C CNN
-	1    4800 4600
-	1    0    0    -1
-$EndComp
-Connection ~ 4800 4600
 Wire Notes Line
 	5200 3850 3400 3850

Commit message: Wire-up MCU
Parts:
- removed R2: R, symbol Device:R
Connections:
- net labels added: +16V, +3V3
- net labels removed: +5V
- wire segments 52 -> 51
Other:
- note added: "r2 = 1800.0\nr1 = 150.0\n1.25 * (1 + r2/r1) + 100e-6 * r2"
- note added: "r2 = 560.0\nr1 = 330.0\n1.25 * (1 + r2/r1) + 100e-6 * r2"
- note removed: "r2 = 1800\nr1 = 150\nv_out = 1.25 * (1 + r2/r1) + 100e-6 * r2"
- note removed: "r2 = 820\nr1 = 270\nv_out = 1.25 * (1 + r2/r1) + 100e-6 * r2"

Commit message: Finalise component values, add decoupling caps
Parts:
- removed J1: Conn_02x04_Top_Bottom_Shielded, symbol Connector_Generic_Shielded:Conn_02x04_Top_Bottom_Shielded
- removed R1: 100R, symbol Device:R
- added C?: 10n/200V, symbol Device:C
- added C?: 0.1u/50V, symbol Device:C
- added C? (x2): 100n, symbol Device:C
- added C?: 10n, symbol Device:C
- added C?: 1u, symbol Device:C
- added C? (x2): 4u7, symbol Device:C
- added D? (x2): NHP220S, symbol Device:D
- added J?: Conn_02x04_Top_Bottom, symbol Connector_Generic:Conn_02x04_Top_Bottom
- added J?: Conn_01x06, symbol Connector_Generic:Conn_01x06
- added R?: 220k, symbol Device:R
- added R? (x2): 10k, symbol Device:R
- C? (x2): value C -> 1u
- C? (x2): value C -> 4u7
- Q1: value Q_NMOS_GSD -> NCV8406A
Connections:
- net labels added: NRST, SPEED_POT_SLIDER, SWCLK, SWDIO
- net labels removed: GNDA, SPPED_POT_SLIDER
- wire segments 51 -> 93
Other:
- note added: "r2 = 820.0\nr1 = 270.0\n1.25 * (1 + r2/r1) + 100e-6 * r2"
- note removed: "r2 = 560.0\nr1 = 330.0\n1.25 * (1 + r2/r1) + 100e-6 * r2"

Commit message: Fix ERC issues
Parts:
- gave numbers to parts that had none: 26
Connections:
- wire segments 93 -> 106
- no-connect marks 0 -> 8

Commit message: Assign capacitors and resistors
Parts:
- C1, C10, C11, C12, C2, C3, C4, C5, C6, C7, C8, C9: footprint (none) -> Capacitor_SMD:C_0603_1608Metric
- R1, R2, R3, R4, R7: footprint (none) -> Resistor_SMD:R_0603_1608Metric
- R5, R6: footprint (none) -> Resistor_SMD:R_0805_2012Metric
Changed lines of the file:
@@
 F 0 "R4" H 2520 3746 50  0000 L CNN
 F 1 "270" H 2520 3655 50  0000 L CNN
-F 2 "" V 2380 3700 50  0001 C CNN
+F 2 "Resistor_SMD:R_0603_1608Metric" V 2380 3700 50  0001 C CNN
 F 3 "~" H 2450 3700 50  0001 C CNN
 	1    2450 3700
@@
 F 0 "R2" H 2120 4096 50  0000 L CNN
 F 1 "820" H 2120 4005 50  0000 L CNN
-F 2 "" V 1980 4050 50  0001 C CNN
+F 2 "Resistor_SMD:R_0603_1608Metric" V 1980 4050 50  0001 C CNN
 F 3 "~" H 2050 4050 50  0001 C CNN
 	1    2050 4050
@@
 F 0 "C2" H 1665 3746 50  0000 L CNN
 F 1 "1u" H 1665 3655 50  0000 L CNN
-F 2 "" H 1588 3550 50  0001 C CNN
+F 2 "Capacitor_SMD:C_0603_1608Metric" H 1588 3550 50  0001 C CNN
 F 3 "~" H 1550 3700 50  0001 C CNN
 	1    1550 3700
@@
 F 0 "C4" H 2865 3746 50  0000 L CNN
 F 1 "4u7" H 2865 3655 50  0000 L CNN
-F 2 "" H 2788 3550 50  0001 C CNN
+F 2 "Capacitor_SMD:C_0603_1608Metric" H 2788 3550 50  0001 C CNN
 F 3 "~" H 2750 3700 50  0001 C CNN
 	1    2750 3700
@@
 F 0 "R3" H 2520 1996 50  0000 L CNN
 F 1 "150" H 2520 1905 50  0000 L CNN
-F 2 "" V 2380 1950 50  0001 C CNN
+F 2 "Resistor_SMD:R_0603_1608Metric" V 2380 1950 50  0001 C CNN
 F 3 "~" H 2450 1950 50  0001 C CNN
 	1    2450 1950
@@
 F 0 "R1" H 2120 2346 50  0000 L CNN
 F 1 "1k8" H 2120 2255 50  0000 L CNN
-F 2 "" V 1980 2300 50  0001 C CNN
+F 2 "Resistor_SMD:R_0603_1608Metric" V 1980 2300 50  0001 C CNN
 F 3 "~" H 2050 2300 50  0001 C CNN
 	1    2050 2300
@@
 F 0 "C1" H 1665 1996 50  0000 L CNN
 F 1 "1u" H 1665 1905 50  0000 L CNN
-F 2 "" H 1588 1800 50  0001 C CNN
+F 2 "Capacitor_SMD:C_0603_1608Metric" H 1588 1800 50  0001 C CNN
 F 3 "~" H 1550 1950 50  0001 C CNN
 	1    1550 1950
@@
 F 0 "C3" H 2865 1996 50  0000 L CNN
 F 1 "4u7" H 2865 1905 50  0000 L CNN
-F 2 "" H 2788 1800 50  0001 C CNN
+F 2 "Capacitor_SMD:C_0603_1608Metric" H 2788 1800 50  0001 C CNN
 F 3 "~" H 2750 1950 50  0001 C CNN
 	1    2750 1950
@@
 F 0 "C12" H 9815 2046 50  0000 L CNN
 F 1 "10n/200V" H 9815 1955 50  0000 L CNN
-F 2 "" H 9738 1850 50  0001 C CNN
+F 2 "Capacitor_SMD:C_0603_1608Metric" H 9738 1850 50  0001 C CNN
 F 3 "~" H 9700 2000 50  0001 C CNN
 	1    9700 2000
@@
 F 0 "R7" V 9893 1800 50  0000 C CNN
 F 1 "220k" V 9984 1800 50  0000 C CNN
-F 2 "" V 10030 1800 50  0001 C CNN
+F 2 "Resistor_SMD:R_0603_1608Metric" V 10030 1800 50  0001 C CNN
 F 3 "~" H 10100 1800 50  0001 C CNN
 	1    10100 1800
@@
 F 0 "C9" H 7615 1646 50  0000 L CNN
 F 1 "0.1u/50V" H 7615 1555 50  0000 L CNN
-F 2 "" H 7538 1450 50  0001 C CNN
+F 2 "Capacitor_SMD:C_0603_1608Metric" H 7538 1450 50  0001 C CNN
 F 3 "~" H 7500 1600 50  0001 C CNN
 	1    7500 1600
@@
 F 0 "R5" H 8120 1646 50  0000 L CNN
 F 1 "10k" H 8120 1555 50  0000 L CNN
-F 2 "" V 7980 1600 50  0001 C CNN
+F 2 "Resistor_SMD:R_0805_2012Metric" V 7980 1600 50  0001 C CNN
 F 3 "~" H 8050 1600 50  0001 C CNN
 	1    8050 1600
@@
 F 0 "C5" H 4065 2396 50  0000 L CNN
 F 1 "100n" H 4065 2305 50  0000 L CNN
-F 2 "" H 3988 2200 50  0001 C CNN
+F 2 "Capacitor_SMD:C_0603_1608Metric" H 3988 2200 50  0001 C CNN
 F 3 "~" H 3950 2350 50  0001 C CNN
 	1    3950 2350
@@
 F 0 "C8" H 4715 1846 50  0000 L CNN
 F 1 "100n" H 4715 1755 50  0000 L CNN
-F 2 "" H 4638 1650 50  0001 C CNN
+F 2 "Capacitor_SMD:C_0603_1608Metric" H 4638 1650 50  0001 C CNN
 F 3 "~" H 4600 1800 50  0001 C CNN
 	1    4600 1800
@@
 F 0 "C7" H 4415 1846 50  0000 L CNN
 F 1 "10n" H 4415 1755 50  0000 L CNN
-F 2 "" H 4338 1650 50  0001 C CNN
+F 2 "Capacitor_SMD:C_0603_1608Metric" H 4338 1650 50  0001 C CNN
 F 3 "~" H 4300 1800 50  0001 C CNN
 	1    4300 1800
@@
 F 0 "C6" H 4115 1846 50  0000 L CNN
 F 1 "1u" H 4115 1755 50  0000 L CNN
-F 2 "" H 4038 1650 50  0001 C CNN
+F 2 "Capacitor_SMD:C_0603_1608Metric" H 4038 1650 50  0001 C CNN
 F 3 "~" H 4000 1800 50  0001 C CNN
 	1    4000 1800
@@
 F 0 "R6" H 8370 1646 50  0000 L CNN
 F 1 "10k" H 8370 1555 50  0000 L CNN
-F 2 "" V 8230 1600 50  0001 C CNN
+F 2 "Resistor_SMD:R_0805_2012Metric" V 8230 1600 50  0001 C CNN
 F 3 "~" H 8300 1600 50  0001 C CNN
 	1    8300 1600
@@
 F 0 "C10" H 9415 3946 50  0000 L CNN
 F 1 "4u7" H 9415 3855 50  0000 L CNN
-F 2 "" H 9338 3750 50  0001 C CNN
+F 2 "Capacitor_SMD:C_0603_1608Metric" H 9338 3750 50  0001 C CNN
 F 3 "~" H 9300 3900 50  0001 C CNN
 	1    9300 3900
@@
 F 0 "C11" H 9765 3946 50  0000 L CNN
 F 1 "4u7" H 9765 3855 50  0000 L CNN
-F 2 "" H 9688 3750 50  0001 C CNN
+F 2 "Capacitor_SMD:C_0603_1608Metric" H 9688 3750 50  0001 C CNN
 F 3 "~" H 9650 3900 50  0001 C CNN
 	1    9650 3900

Commit message: Add ATB3225, assign all footprints
Parts:
- removed J2: Conn_02x04_Top_Bottom, symbol Connector_Generic:Conn_02x04_Top_Bottom
- removed U1, U3: LM317_3PinPackage, symbol Regulator_Linear:LM317_3PinPackage
- added J2: Conn_02x04_Odd_Even, Connector_PinSocket_2.54mm:PinSocket_2x04_P2.54mm_Vertical, symbol Connector_Generic:Conn_02x04_Odd_Even
- added U1, U3: LM317L_SO8, Package_SO:SOIC-8_3.9x4.9mm_P1.27mm, symbol Regulator_Linear:LM317L_SO8
- D1, D2: footprint (none) -> Diode_SMD:D_SOD-123F
- J1: footprint (none) -> Connector_PinHeader_2.54mm:PinHeader_1x06_P2.54mm_Vertical
- J3: footprint (none) -> Connector_PinSocket_2.54mm:PinSocket_1x02_P2.54mm_Vertical
- Q1: footprint (none) -> Package_TO_SOT_SMD:SOT-223
- TR1: value ATB3225 -> ATB322524-0110; footprint (none) -> speedctrl-footprints:ATB3225
Changed lines of the file:
@@
 	8500 3750 8500 3650
-$Comp
-L Regulator_Linear:LM317_3PinPackage U3
-U 1 1 5BB14FB2
-P 2050 3550
-F 0 "U3" H 2050 3792 50  0000 C CNN
-F 1 "LM317_3PinPackage" H 2050 3701 50  0000 C CNN
-F 2 "" H 2050 3800 50  0001 C CIN
-F 3 "http://www.ti.com/lit/ds/symlink/lm317.pdf" H 2050 3550 50  0001 C CNN
-	1    2050 3550
-	1    0    0    -1
-$EndComp
 $Comp
 L speedctrl_parts:ATB3225 TR1
@@
 P 8900 2000
 F 0 "TR1" H 8900 2425 50  0000 C CNN
-F 1 "ATB3225" H 8900 2334 50  0000 C CNN
-F 2 "" H 8700 1750 50  0001 C CNN
+F 1 "ATB322524-0110" H 8900 2334 50  0000 C CNN
+F 2 "speedctrl-footprints:ATB3225" H 8700 1750 50  0001 C CNN
 F 3 "" H 8700 1750 50  0001 C CNN
 	1    8900 2000
@@
 F 0 "Q1" H 8605 2646 50  0000 L CNN
 F 1 "NCV8406A" H 8605 2555 50  0000 L CNN
-F 2 "" H 8600 2700 50  0001 C CNN
+F 2 "Package_TO_SOT_SMD:SOT-223" H 8600 2700 50  0001 C CNN
 F 3 "https://www.onsemi.com/pub/Collateral/NCV8406-D.PDF" H 8400 2600 50  0001 C CNN
 	1    8400 2600
@@
 F 0 "J3" H 10730 1792 50  0000 L CNN
 F 1 "Conn_01x02" H 10730 1701 50  0000 L CNN
-F 2 "" H 10650 1800 50  0001 C CNN
+F 2 "Connector_PinSocket_2.54mm:PinSocket_1x02_P2.54mm_Vertical" H 10650 1800 50  0001 C CNN
 F 3 "~" H 10650 1800 50  0001 C CNN
 	1    10650 1800
@@
 Wire Wire Line
 	2050 3850 2050 3900
-Connection ~ 2050 3850
 Wire Wire Line
 	2450 3550 2350 3550
@@
 	1550 3550 1750 3550
 $Comp
-L Regulator_Linear:LM317_3PinPackage U1
-U 1 1 5BC29C63
-P 2050 1800
-F 0 "U1" H 2050 2042 50  0000 C CNN
-F 1 "LM317_3PinPackage" H 2050 1951 50  0000 C CNN
-F 2 "" H 2050 2050 50  0001 C CIN
-F 3 "http://www.ti.com/lit/ds/symlink/lm317.pdf" H 2050 1800 50  0001 C CNN
-	1    2050 1800
-	1    0    0    -1
-$EndComp
-$Comp
 L power:+24V #PWR0109
 U 1 1 5BC29C6A
@@
 Wire Wire Line
 	2050 2100 2050 2150
-Connection ~ 2050 2100
 Wire Wire Line
 	2450 1800 2350 1800
@@
 Connection ~ 10450 2200
 $Comp
-L Connector_Generic:Conn_02x04_Top_Bottom J2
-U 1 1 5C2B3B9E
-P 8500 5400
-F 0 "J2" H 8550 5717 50  0000 C CNN
-F 1 "Conn_02x04_Top_Bottom" H 8550 5626 50  0000 C CNN
-F 2 "" H 8500 5400 50  0001 C CNN
-F 3 "~" H 8500 5400 50  0001 C CNN
-	1    8500 5400
-	1    0    0    -1
-$EndComp
-$Comp
 L Device:C C9
 U 1 1 5C2B752B
@@
 F 0 "J1" H 6430 3592 50  0000 L CNN
 F 1 "Conn_01x06" H 6430 3501 50  0000 L CNN
-F 2 "" H 6350 3600 50  0001 C CNN
+F 2 "Connector_PinHeader_2.54mm:PinHeader_1x06_P2.54mm_Vertical" H 6350 3600 50  0001 C CNN
 F 3 "~" H 6350 3600 50  0001 C CNN
 	1    6350 3600
@@
 F 0 "D2" H 9500 1584 50  0000 C CNN
 F 1 "NHP220S" H 9500 1675 50  0000 C CNN
-F 2 "" H 9500 1800 50  0001 C CNN
+F 2 "Diode_SMD:D_SOD-123F" H 9500 1800 50  0001 C CNN
 F 3 "~" H 9500 1800 50  0001 C CNN
 	1    9500 1800
@@
 F 0 "D1" V 7454 2079 50  0000 L CNN
 F 1 "NHP220S" V 7545 2079 50  0000 L CNN
-F 2 "" H 7500 2000 50  0001 C CNN
+F 2 "Diode_SMD:D_SOD-123F" H 7500 2000 50  0001 C CNN
 F 3 "~" H 7500 2000 50  0001 C CNN
 	1    7500 2000
@@
 L power:GND #PWR0122
 U 1 1 5C50B6D9
-P 8800 5700
-F 0 "#PWR0122" H 8800 5450 50  0001 C CNN
-F 1 "GND" H 8805 5527 50  0000 C CNN
-F 2 "" H 8800 5700 50  0001 C CNN
-F 3 "" H 8800 5700 50  0001 C CNN
-	1    8800 5700
-	1    0    0    -1
-$EndComp
-Wire Wire Line
-	8800 5500 8800 5600
-Connection ~ 8800 5600
-Wire Wire Line
-	8800 5600 8800 5700
+P 9150 5600
+F 0 "#PWR0122" H 9150 5350 50  0001 C CNN
+F 1 "GND" H 9155 5427 50  0000 C CNN
+F 2 "" H 9150 5600 50  0001 C CNN
+F 3 "" H 9150 5600 50  0001 C CNN
+	1    9150 5600
+	1    0    0    -1
+$EndComp
 Wire Wire Line
 	6900 5400 8300 5400
@@
 Wire Wire Line
 	1900 5300 1900 5000
+$Comp
+L Regulator_Linear:LM317L_SO8 U1
+U 1 1 5C5F4905
+P 2050 1800
+F 0 "U1" H 2050 2042 50  0000 C CNN
+F 1 "LM317L_SO8" H 2050 1951 50  0000 C CNN
+F 2 "Package_SO:SOIC-8_3.9x4.9mm_P1.27mm" H 2050 2000 50  0001 C CIN
+F 3 "http://www.ti.com/lit/ds/snvs775k/snvs775k.pdf" H 2050 1600 50  0001 C CNN
+	1    2050 1800
+	1    0    0    -1
+$EndComp
+Connection ~ 2050 2100
+$Comp
+L Regulator_Linear:LM317L_SO8 U3
+U 1 1 5C5F49A9
+P 2050 3550
+F 0 "U3" H 2050 3792 50  0000 C CNN
+F 1 "LM317L_SO8" H 2050 3701 50  0000 C CNN
+F 2 "Package_SO:SOIC-8_3.9x4.9mm_P1.27mm" H 2050 3750 50  0001 C CIN
+F 3 "http://www.ti.com/lit/ds/snvs775k/snvs775k.pdf" H 2050 3350 50  0001 C CNN
+	1    2050 3550
+	1    0    0    -1
+$EndComp
+Connection ~ 2050 3850
+Wire Wire Line
+	8800 5500 8800 5600
+$Comp
+L Connector_Generic:Conn_02x04_Odd_Even J2
+U 1 1 5C5FBB0B
+P 8600 5500
+F 0 "J2" H 8650 5817 50  0000 C CNN
+F 1 "Conn_02x04_Odd_Even" H 8650 5726 50  0000 C CNN
+F 2 "Connector_PinSocket_2.54mm:PinSocket_2x04_P2.54mm_Vertical" H 8600 5500 50  0001 C CNN
+F 3 "~" H 8600 5500 50  0001 C CNN
+	1    8600 5500
+	-1   0    0    1
+$EndComp
+Wire Wire Line
+	8800 5600 9150 5600
+Connection ~ 8800 5600
 $EndSCHEMATC

Commit message: Replace pin sockets with header footprints
Parts:
- J2: footprint Connector_PinSocket_2.54mm:PinSocket_2x04_P2.54mm_Vertical -> Connector_PinHeader_2.54mm:PinHeader_2x04_P2.54mm_Vertical
- J3: footprint Connector_PinSocket_2.54mm:PinSocket_1x02_P2.54mm_Vertical -> Connector_PinHeader_2.54mm:PinHeader_1x02_P2.54mm_Vertical
Changed lines of the file:
@@
 F 0 "J3" H 10730 1792 50  0000 L CNN
 F 1 "Conn_01x02" H 10730 1701 50  0000 L CNN
-F 2 "Connector_PinSocket_2.54mm:PinSocket_1x02_P2.54mm_Vertical" H 10650 1800 50  0001 C CNN
+F 2 "Connector_PinHeader_2.54mm:PinHeader_1x02_P2.54mm_Vertical" H 10650 1800 50  0001 C CNN
 F 3 "~" H 10650 1800 50  0001 C CNN
 	1    10650 1800
@@
 F 0 "J2" H 8650 5817 50  0000 C CNN
 F 1 "Conn_02x04_Odd_Even" H 8650 5726 50  0000 C CNN
-F 2 "Connector_PinSocket_2.54mm:PinSocket_2x04_P2.54mm_Vertical" H 8600 5500 50  0001 C CNN
+F 2 "Connector_PinHeader_2.54mm:PinHeader_2x04_P2.54mm_Vertical" H 8600 5500 50  0001 C CNN
 F 3 "~" H 8600 5500 50  0001 C CNN
 	1    8600 5500

Commit message: Initial part placement
Parts:
- removed Q1: NCV8406A, Package_TO_SOT_SMD:SOT-223, symbol Device:Q_NMOS_GSD
- added Q1: Q_NMOS_GDSD, Package_TO_SOT_SMD:SOT-223, symbol Device:Q_NMOS_GDSD
Connections:
- wire segments 106 -> 109
Changed lines of the file:
@@
-$EndComp
-$Comp
-L Device:Q_NMOS_GSD Q1
-U 1 1 5BB5835D
-P 8400 2600
-F 0 "Q1" H 8605 2646 50  0000 L CNN
-F 1 "NCV8406A" H 8605 2555 50  0000 L CNN
-F 2 "Package_TO_SOT_SMD:SOT-223" H 8600 2700 50  0001 C CNN
-F 3 "https://www.onsemi.com/pub/Collateral/NCV8406-D.PDF" H 8400 2600 50  0001 C CNN
-	1    8400 2600
-	1    0    0    -1
 $EndComp
 $Comp
@@
 $EndComp
 Wire Wire Line
-	8500 2200 8500 2400
+	8500 2200 8500 2300
 Wire Wire Line
 	7500 1400 7500 1450
@@
 	8800 5600 9150 5600
 Connection ~ 8800 5600
+$Comp
+L Device:Q_NMOS_GDSD Q1
+U 1 1 5C6155B0
+P 8400 2600
+F 0 "Q1" H 8687 2646 50  0000 L CNN
+F 1 "Q_NMOS_GDSD" H 8687 2555 50  0000 L CNN
+F 2 "Package_TO_SOT_SMD:SOT-223" H 8600 2700 50  0001 C CNN
+F 3 "~" H 8400 2600 50  0001 C CNN
+	1    8400 2600
+	1    0    0    -1
+$EndComp
+Wire Wire Line
+	8600 2400 8600 2300
+Wire Wire Line
+	8600 2300 8500 2300
+Connection ~ 8500 2300
+Wire Wire Line
+	8500 2300 8500 2400
 $EndSCHEMATC
