File: speedctrl.sch (KiCad schematic (older format))
At the start: 30 parts, among them J1 Conn_01x06, J2 Conn_02x04_Odd_Even, J3 Conn_01x02, Q1 Q_NMOS_GDSD, U1 LM317L_SO8, U2 BD6231, U3 LM317L_SO8, U4 STM32F030F4Px

Commit message: Add crystal and mounting holes
Parts:
- added C13, C14: 10pF, Capacitor_SMD:C_0603_1608Metric, symbol Device:C
- added H1, H2, H3, H4: MountingHole, MountingHole:MountingHole_3.2mm_M3, symbol Mechanical:MountingHole
- added Y1: ABM10-16MHz, Crystal:Crystal_SMD_Abracon_ABM10-4Pin_2.5x2.0mm, symbol Device:Crystal
Connections:
- wire segments 109 -> 117
- no-connect marks 8 -> 6
Changed lines of the file:
@@
 	4450 2500 3950 2500
 Connection ~ 3950 2500
-Wire Wire Line
-	3950 2200 3650 2200
-Wire Wire Line
-	3650 2200 3650 3800
-Wire Wire Line
-	3650 3800 6150 3800
 Connection ~ 3950 2200
 Text Label 5850 3800 0    50   ~ 0
@@
 U 1 1 5C2E5320
 P 4000 1800
-F 0 "C6" H 4115 1846 50  0000 L CNN
-F 1 "1u" H 4115 1755 50  0000 L CNN
+F 0 "C6" H 3885 1846 50  0000 R CNN
+F 1 "1u" H 3885 1755 50  0000 R CNN
 F 2 "Capacitor_SMD:C_0603_1608Metric" H 4038 1650 50  0001 C CNN
 F 3 "~" H 4000 1800 50  0001 C CNN
@@
 NoConn ~ 5450 2500
 NoConn ~ 5450 2700
-NoConn ~ 4450 3000
-NoConn ~ 4450 3100
 NoConn ~ 4450 3300
 $Comp
@@
 U 1 1 5C5FBB0B
 P 8600 5500
-F 0 "J2" H 8650 5817 50  0000 C CNN
-F 1 "Conn_02x04_Odd_Even" H 8650 5726 50  0000 C CNN
+F 0 "J2" H 8650 5075 50  0000 C CNN
+F 1 "Conn_02x04_Odd_Even" H 8650 5166 50  0000 C CNN
 F 2 "Connector_PinHeader_2.54mm:PinHeader_2x04_P2.54mm_Vertical" H 8600 5500 50  0001 C CNN
 F 3 "~" H 8600 5500 50  0001 C CNN
@@
 Wire Wire Line
 	8500 2300 8500 2400
+$Comp
+L Device:Crystal Y1
+U 1 1 5C61C680
+P 3900 3150
+F 0 "Y1" V 3854 3281 50  0000 L CNN
+F 1 "ABM10-16MHz" H 3945 3281 50  0000 L BNN
+F 2 "Crystal:Crystal_SMD_Abracon_ABM10-4Pin_2.5x2.0mm" H 3900 3150 50  0001 C CNN
+F 3 "~" H 3900 3150 50  0001 C CNN
+	1    3900 3150
+	0    -1   -1   0
+$EndComp
+Wire Wire Line
+	4450 3000 3900 3000
+Wire Wire Line
+	4450 3100 4350 3100
+Wire Wire Line
+	4350 3100 4350 3300
+Wire Wire Line
+	4350 3300 3900 3300
+Wire Wire Line
+	3250 2200 3250 3800
+Wire Wire Line
+	3250 2200 3950 2200
+Wire Wire Line
+	3250 3800 6150 3800
+$Comp
+L Device:C C13
+U 1 1 5C651F13
+P 3600 3000
+F 0 "C13" V 3348 3000 50  0000 C CNN
+F 1 "10pF" V 3439 3000 50  0000 C CNN
+F 2 "Capacitor_SMD:C_0603_1608Metric" H 3638 2850 50  0001 C CNN
+F 3 "~" H 3600 3000 50  0001 C CNN
+	1    3600 3000
+	0    1    1    0
+$EndComp
+$Comp
+L Device:C C14
+U 1 1 5C651FEA
+P 3600 3300
+F 0 "C14" V 3348 3300 50  0000 C CNN
+F 1 "10pF" V 3439 3300 50  0000 C CNN
+F 2 "Capacitor_SMD:C_0603_1608Metric" H 3638 3150 50  0001 C CNN
+F 3 "~" H 3600 3300 50  0001 C CNN
+	1    3600 3300
+	0    1    1    0
+$EndComp
+$Comp
+L power:GND #PWR03
+U 1 1 5C65207C
+P 3450 3450
+F 0 "#PWR03" H 3450 3200 50  0001 C CNN
+F 1 "GND" H 3455 3277 50  0000 C CNN
+F 2 "" H 3450 3450 50  0001 C CNN
+F 3 "" H 3450 3450 50  0001 C CNN
+	1    3450 3450
+	1    0    0    -1
+$EndComp
+Wire Wire Line
+	3450 3450 3450 3300
+Connection ~ 3450 3300
+Wire Wire Line
+	3450 3300 3450 3000
+Wire Wire Line
+	3750 3300 3900 3300
+Connection ~ 3900 3300
+Wire Wire Line
+	3750 3000 3900 3000
+Connection ~ 3900 3000
+$Comp
+L Mechanical:MountingHole H1
+U 1 1 5C662D45
+P 3050 5250
+F 0 "H1" H 3150 5296 50  0000 L CNN
+F 1 "MountingHole" H 3150 5205 50  0000 L CNN
+F 2 "MountingHole:MountingHole_3.2mm_M3" H 3050 5250 50  0001 C CNN
+F 3 "~" H 3050 5250 50  0001 C CNN
+	1    3050 5250
+	1    0    0    -1
+$EndComp
+$Comp
+L Mechanical:MountingHole H2
+U 1 1 5C662DC1
+P 3050 5500
+F 0 "H2" H 3150 5546 50  0000 L CNN
+F 1 "MountingHole" H 3150 5455 50  0000 L CNN
+F 2 "MountingHole:MountingHole_3.2mm_M3" H 3050 5500 50  0001 C CNN
+F 3 "~" H 3050 5500 50  0001 C CNN
+	1    3050 5500
+	1    0    0    -1
+$EndComp
+$Comp
+L Mechanical:MountingHole H3
+U 1 1 5C662E2F
+P 3050 5750
+F 0 "H3" H 3150 5796 50  0000 L CNN
+F 1 "MountingHole" H 3150 5705 50  0000 L CNN
+F 2 "MountingHole:MountingHole_3.2mm_M3" H 3050 5750 50  0001 C CNN
+F 3 "~" H 3050 5750 50  0001 C CNN
+	1    3050 5750
+	1    0    0    -1
+$EndComp
+$Comp
+L Mechanical:MountingHole H4
+U 1 1 5C662EAF
+P 3050 6000
+F 0 "H4" H 3150 6046 50  0000 L CNN
+F 1 "MountingHole" H 3150 5955 50  0000 L CNN
+F 2 "MountingHole:MountingHole_3.2mm_M3" H 3050 6000 50  0001 C CNN
+F 3 "~" H 3050 6000 50  0001 C CNN
+	1    3050 6000
+	1    0    0    -1
+$EndComp
 $EndSCHEMATC

Commit message: Use DRV8816 instead of the original driver, use BSS138 for flyback
Parts:
- removed J1: Conn_01x06, Connector_PinHeader_2.54mm:PinHeader_1x06_P2.54mm_Vertical, symbol Connector_Generic:Conn_01x06
- removed Q1: Q_NMOS_GDSD, Package_TO_SOT_SMD:SOT-223, symbol Device:Q_NMOS_GDSD
- removed U1, U3: LM317L_SO8, Package_SO:SOIC-8_3.9x4.9mm_P1.27mm, symbol Regulator_Linear:LM317L_SO8
- removed U2: BD6231, Package_SO:SSOP-8_3.95x5.21x3.27mm_P1.27mm, symbol speedctrl_parts:BD6231
- removed U4: STM32F030F4Px, Package_SO:TSSOP-20_4.4x6.5mm_P0.65mm, symbol MCU_ST_STM32F0:STM32F030F4Px
- removed Y1: ABM10-16MHz, Crystal:Crystal_SMD_Abracon_ABM10-4Pin_2.5x2.0mm, symbol Device:Crystal
- added C15: 100n, Capacitor_SMD:C_0603_1608Metric, symbol Device:C
- added D3: HSMY-C170, LED_SMD:LED_0805_2012Metric_Pad1.15x1.40mm_HandSolder, symbol Device:LED
- added D4: HSMG-C170, LED_SMD:LED_0805_2012Metric_Pad1.15x1.40mm_HandSolder, symbol Device:LED
- added J1: Conn_01x05, Connector_PinHeader_2.54mm:PinHeader_1x05_P2.54mm_Vertical, symbol Connector_Generic:Conn_01x05
- added Q1: BSS138, Package_TO_SOT_SMD:SOT-23, symbol Transistor_FET:BSS138
- added R8: 10k, Resistor_SMD:R_0603_1608Metric, symbol Device:R
- added U1: LM317_3PinPackage, Package_TO_SOT_SMD:SOT-223-3_TabPin2, symbol Regulator_Linear:LM317_3PinPackage
- added U2: DRV8816PWPR, Package_SO:HTSSOP-16-1EP_4.4x5mm_P0.65mm_EP3.4x5mm_Mask2.46x2.31mm_ThermalVias, symbol speedctrl_parts:DRV8816PWPR
- added U3: STM32F070F6Px, Package_SO:TSSOP-20_4.4x6.5mm_P0.65mm, symbol MCU_ST_STM32F0:STM32F070F6Px
- added Y1: Crystal_GND24, Crystal:Crystal_SMD_Abracon_ABM10-4Pin_2.5x2.0mm, symbol Device:Crystal_GND24
- C1: value 1u -> 100n
- C12: footprint Capacitor_SMD:C_0603_1608Metric -> Capacitor_SMD:C_1206_3216Metric
- C3: value 4u7 -> 100n
- D1, D2: value NHP220S -> DA2JF8100L; footprint Diode_SMD:D_SOD-123F -> speedctrl-footprints:Diode_SMini2-F5-B
- H1, H2, H3, H4: footprint MountingHole:MountingHole_3.2mm_M3 -> MountingHole:MountingHole_2.2mm_M2
- J2: footprint Connector_PinHeader_2.54mm:PinHeader_2x04_P2.54mm_Vertical -> Connector_IDC:IDC-Header_2x04_P2.54mm_Vertical
- R1: value 1k8 -> 330
- R2: value 820 -> 560
- R3: value 150 -> 330
- R4: value 270 -> 330
- R7: footprint Resistor_SMD:R_0603_1608Metric -> Resistor_SMD:R_0805_2012Metric
Connections:
- net labels removed: +16V, NRST
- wire segments 117 -> 133
- no-connect marks 6 -> 7
Other:
- note added: "r2 = 560.0\nr1 = 330.0\n1.25 * (1 + r2/r1) + 100e-6 * r2"
- note removed: "r2 = 1800.0\nr1 = 150.0\n1.25 * (1 + r2/r1) + 100e-6 * r2"
- note removed: "r2 = 820.0\nr1 = 270.0\n1.25 * (1 + r2/r1) + 100e-6 * r2"
